File: USB2CAN.kicad_pcb (KiCad board)
At the start: 2 copper layers, 53.3 x 44.9 mm, 94 parts, among them J1 Conn_01x04, J2 Conn_01x02, J3 Conn_01x02, J4 Conn_01x02, J5 Conn_01x02, U1 HX9193, U10 SL2.1S, U2 STM32F072C8Tx, U3 TJA1051T-3, U4 STM32F072C8Tx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

Commit message: Add ESD protection
Parts:
- added D13: BV03C, Diode_SMD:D_SOD-323, F.Cu at (84.5, 35.5)
- added U11: ~, Package_TO_SOT_SMD:SOT-23-3, F.Cu at (87.7, 62.1)
- added U12: ~, Package_TO_SOT_SMD:SOT-23-3, F.Cu at (88.1, 34.2)
- added U13: ~, Package_TO_SOT_SMD:SOT-23-3, F.Cu at (128.7, 34.2)
- added U14: ~, Package_TO_SOT_SMD:SOT-23-3, F.Cu at (128.8, 62.0)
- moved C19 5.41 mm to (89.1, 38.3), turned to -90 degrees
- moved C36 3.99 mm to (83.8, 42.1), turned to 180 degrees
- moved D1 2.14 mm to (84.4, 57.2)
- moved R1 2.14 mm to (86.5, 57.3)
- moved C15 2.06 mm to (88.6, 57.3)
- moved C25 2.01 mm to (127.8, 37.8), turned to 90 degrees
- moved U1 1.53 mm to (86.5, 38.9)
- moved C28 1.17 mm to (86.8, 42.1)
- moved C40 0.48 mm to (99.3, 47.2)
- moved C39 0.37 mm to (99.3, 50.3)
- moved C2 0.33 mm to (89.1, 41.3)
- moved C6 0.31 mm to (106.9, 42.5)
- moved C35 0.27 mm to (117.5, 51.4), turned to 90 degrees
- moved C1 0.17 mm to (124.1, 43.6)
- moved C26 0.07 mm to (97.5, 42.5), turned to 180 degrees
Routing:
- net /STM2_CAN/CAN_L: track 6.57 -> 16.5 mm
- net /STM_CAN3/CAN_H: track 6.53 -> 16.2 mm
- net /STM1_CAN/CAN_H: track 7.59 -> 16.4 mm
- net /STM_CAN4/CAN_L: track 6.90 -> 15.3 mm
- net VCC: track 266.3 -> 274.2 mm
- net /STM1_CAN/CAN_L: track 6.87 -> 13.8 mm
- net /STM2_CAN/CAN_H: track 6.24 -> 13.1 mm
- net /STM_CAN3/CAN_L: track 6.24 -> 13.1 mm
- net /STM_CAN4/CAN_H: track 6.80 -> 11.2 mm
- net +5V: track 98.9 -> 96.7 mm
- net Net-(U10-VDD33): track 2.11 -> 2.96 mm
- net /STM1_CAN/CAN_RX: track 21.1 -> 20.3 mm
- net /USB_HUB/XIN: track 4.48 -> 5.11 mm
- net GND: track 16.9 -> 16.4 mm, vias 20 -> 33
Other:
- board text added: "0"
- board text added: "10K"
- board text added: "18p"
