File: subsch/STM1_CAN.kicad_sch (KiCad schematic)
At the start: 17 parts

Commit message: Add ESD protection
Parts:
- added U11: ~, Package_TO_SOT_SMD:SOT-23-3, symbol Extra IC:PESD1CAN
- C13, C14, C15, C16, C17, C18, C19, C20: value (none) -> 100n; footprint (none) -> Capacitor_SMD:C_0603_1608Metric
- D7, D8: value (none) -> LED; footprint (none) -> LED_SMD:LED_0603_1608Metric
- R10, R9: value (none) -> 1K; footprint (none) -> Resistor_SMD:R_0603_1608Metric
- R11: value (none) -> 120; footprint (none) -> Resistor_SMD:R_0603_1608Metric
- R7: value (none) -> 0; footprint (none) -> Resistor_SMD:R_0603_1608Metric
- R8: value (none) -> 10K; footprint (none) -> Resistor_SMD:R_0603_1608Metric
- U4: value (none) -> STM32F072C8Tx; footprint (none) -> Package_QFP:LQFP-48_7x7mm_P0.5mm
- U5: value (none) -> TJA1051T-3; footprint (none) -> Package_SO:SOIC-8_3.9x4.9mm_P1.27mm
Connections:
- net CAN_H: now also U11.1 (H)
- net CAN_L: now also U11.2 (L)
- net GND: now also U11.3 (GND)
