File: subsch/STM3_CAN.kicad_sch (KiCad schematic)
At the start: 17 parts

Commit message: Add ESD protection
Parts:
- added U12: ~, Package_TO_SOT_SMD:SOT-23-3, symbol Extra IC:PESD1CAN
- C29, C30, C31, C32, C33, C34, C35, C36: value (none) -> 100n; footprint (none) -> Capacitor_SMD:C_0603_1608Metric
- D11, D12: value (none) -> LED; footprint (none) -> LED_SMD:LED_0603_1608Metric
- R17: value (none) -> 0; footprint (none) -> Resistor_SMD:R_0603_1608Metric
- R18: value (none) -> 10K; footprint (none) -> Resistor_SMD:R_0603_1608Metric
- R19, R20: value (none) -> 1K; footprint (none) -> Resistor_SMD:R_0603_1608Metric
- R21: value (none) -> 120; footprint (none) -> Resistor_SMD:R_0603_1608Metric
- U8: value (none) -> STM32F072C8Tx; footprint (none) -> Package_QFP:LQFP-48_7x7mm_P0.5mm
- U9: value (none) -> TJA1051T-3; footprint (none) -> Package_SO:SOIC-8_3.9x4.9mm_P1.27mm
Connections:
- net CAN_H: now also U12.1 (H)
- net CAN_L: now also U12.2 (L)
- net GND: now also U12.3 (GND)
