File: subsch/STM4_CAN.kicad_sch (KiCad schematic)
At the start: 17 parts

Commit message: Add ESD protection
Parts:
- added U12: ~, Package_TO_SOT_SMD:SOT-23-3, symbol Extra IC:PESD1CAN
- C21, C22, C23, C24, C25, C26, C27, C28: value (none) -> 100n; footprint (none) -> Capacitor_SMD:C_0603_1608Metric
- D10, D9: value (none) -> LED; footprint (none) -> LED_SMD:LED_0603_1608Metric
- R12: value (none) -> 0; footprint (none) -> Resistor_SMD:R_0603_1608Metric
- R13: value (none) -> 10K; footprint (none) -> Resistor_SMD:R_0603_1608Metric
- R14, R15: value (none) -> 1K; footprint (none) -> Resistor_SMD:R_0603_1608Metric
- R16: value (none) -> 120; footprint (none) -> Resistor_SMD:R_0603_1608Metric
- U6: value (none) -> STM32F072C8Tx; footprint (none) -> Package_QFP:LQFP-48_7x7mm_P0.5mm
- U7: value (none) -> TJA1051T-3; footprint (none) -> Package_SO:SOIC-8_3.9x4.9mm_P1.27mm
Connections:
- net CAN_H: now also U12.1 (H)
- net CAN_L: now also U12.2 (L)
- net GND: now also U12.3 (GND)
